File: SDC.kicad_sch (KiCad schematic)
At the start: 0 parts

Commit message: Had not saved changes, this commit is for the last one :)
Parts:
- added B1: COCKPIT, symbol FSUK_ADS:NC_BUTTON
- added B2: LEFT, symbol FSUK_ADS:NC_BUTTON
- added B3: RIGHT, symbol FSUK_ADS:NC_BUTTON
- added BT2: +12V, symbol Device:Battery
- added C1: BSPD, symbol FSUK_ADS:BSPD
- added D1, D2, D3, D4, D5: LED, symbol Device:LED
- added F12: BOTS, symbol FSUK_ADS:BOTS
- added F13: 80 A, symbol Device:Fuse
- added F14: INERTIA_SW, symbol FSUK_ADS:INERTIA
- added K1: SW80, symbol FSUK_ADS:SW80_Contactor
- added K2: SISF2, symbol FSUK_ADS:SISF2
- added K3: COMPUTE, symbol FSUK_ADS:RELAY_COMP_SPDT
- added K4: AS CONTACTOR, symbol FSUK_ADS:POWER_RELAY_MKS_DPDT
- added M1: LVMS, symbol FSUK_ADS:LVMS
- added M2: ASMS, symbol FSUK_ADS:ASMS
- added RES1: RES CONTACTOR, symbol FSUK_ADS:Remote_Emergency_Stop
- added SW1: COMPUTE_SW, symbol FSUK_ADS:SW_COMPUTE
- added V3: 12->24V, symbol FSUK_ADS:Voltage_Converter
Connections:
- new net: F13.1, M1.1 (IN)
- new net: K4.4 (NC), RES1.SI2-3 (SDC_OUT)
- new net: BT2.1 (+), F13.2
- new net: C1.2 (RLY_OUT), D5.2 (A)
- new net BYPASS: B3.2 (OUT), K2.12 (IN), RES1.SI2-1 (SDC_IN)
- new net COIL_24V_ASMS: K2.24 (IN), K2.A2 (+), V3.3 (VOUT+)
- new net COIL_24V_SW80_ASMS: K1.A2 (+), K2.23 (OUT)
- new net COIL_COMPUTE: K3.86 (+), SW1.2 (OUT)
- new net GND_IC: BT2.2 (-), C1.4 (GND), D1.1 (K), D2.1 (K), D3.1 (K), D4.1 (K), D5.1 (K), K1.A1 (-), K2.A1 (-), K3.85 (-), V3.2 (GND), V3.4 (GND)
- new net SDC_1: B1.2 (OUT), B2.1 (IN)
- new net SDC_2: B2.2 (OUT), B3.1 (IN)
- new net SDC_3: D2.2 (A), F12.1 (IN), K2.11 (OUT), K4.1 (IN)
- new net SDC_4: D3.2 (A), F12.2 (OUT), F14.1 (IN)
- new net SDC_5: C1.1 (RLY_IN), C1.3 (VIN), D4.2 (A), F14.2 (OUT)
- new net SDC_SPINE: B1.1 (IN), D1.2 (A), M1.2 (OUT), M2.1 (IN), SW1.1 (IN)
- new net SDC_SPINE_ASMS: M2.2 (OUT), V3.1 (VIN+)
Other:
- note added: "Coil for SW80 contactor on ADS_Power_Circuit page. Switched by LVMS/ASMS/RES Bypass path. (T14.5.4 & T14.3.5)"
- note added: "EBS stuff needs to go here!"
- note added: "Gates compute module on ADS page. Compute switched by LVMS."
- note added: "Manual Toggle"
- note added: "T14.3.5 Forcibly guided"
- title: (none) -> ADS Shutdown Circuit
