File: kiCad/fsuk-ads-electrical/ads_power_circuit.kicad_sch (KiCad schematic)
At the start: 16 parts, among them K1 SW80, K3 COMPUTE

Commit message: Added documentation to try describe some things
Other:
- note added: "Barrel Jack for both."
- note added: "USB-C connection via breakout."
Changed lines of the file:
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@@
+		)
+	)
+	(text "USB-C connection\nvia breakout.\n"
+		(exclude_from_sim no)
+		(at 99.822 146.05 0)
+		(effects
+			(font
+				(size 1.27 1.27)
+			)
 		)
 	)
@@
 		(effects
 			(font
+				(size 1.27 1.27)
+			)
+		)
+	)
+	(text "Barrel Jack\nfor both.\n"
+		(exclude_from_sim no)
+		(at 61.722 147.32 0)
+		(effects
+			(font
